File: STM32L475-protoboard.kicad_pcb (KiCad board)
At the start: 2 copper layers, 84.9 x 52.9 mm, 44 parts, among them J1 USB_HEADER, J10 Conn_01x01_Female, J2 USB_B_Micro, J3 STLINK, J4 W5500_ETHERNET, J6 Conn_01x20_Male, J7 Conn_01x20_Male, J8 Conn_01x01_Female, J9 Conn_01x01_Female, SW1 RESET, U1 SRV05-4, U2 AMS1117-3.3, U3 STM32L475RCTx, Y1 Crystal_GND24

Commit message: final commit for this session, to be continued
Parts:
- added J6: Conn_01x02_Male, Connector_PinHeader_2.54mm:PinHeader_1x02_P2.54mm_Vertical, F.Cu at (145.8, 66.3)
- added JP1: J, Jumper:SolderJumper-2_P1.3mm_Open_RoundedPad1.0x1.5mm, F.Cu at (143.6, 61.7)
- moved R1 3.80 mm to (139.2, 61.7)
- renumbered J9 to J10, J10 to J11, J4 to J5, J6 to J7, J7 to J8, J8 to J9
Connections:
- R1 pad 2: Net-(D2-Pad2) -> Net-(R1-Pad2)
Routing:
- net Net-(R1-Pad2): track 0.00 -> 7.53 mm
- net GND: track 46.5 -> 48.7 mm, vias 87 -> 88

Commit message: save
Parts:
- added J10: Conn_01x02_Male, Connector_PinHeader_2.54mm:PinHeader_1x02_P2.54mm_Vertical, F.Cu at (143.5, 91.4)
- added J6: JST_BATT, Connector_PinHeader_2.54mm:PinHeader_1x02_P2.54mm_Vertical, F.Cu at (71.1, 64.3)
- added J7: BOOT_MODE, Connector_PinHeader_2.54mm:PinHeader_1x03_P2.54mm_Vertical, F.Cu at (105.2, 89.9)
- added JP2: J, Jumper:SolderJumper-2_P1.3mm_Open_RoundedPad1.0x1.5mm, F.Cu at (141.6, 95.2)
- added R2: 10k, Resistor_SMD:R_0603_1608Metric_Pad0.98x0.95mm_HandSolder, F.Cu at (105.0, 92.8)
- J14: renamed from J8; value Conn_01x20_Male -> lower_header
- J8: renamed from J7; value Conn_01x20_Male -> upper_header
- moved J3 46.4 mm to (85.8, 101.2), turned to -90 degrees
- moved J13 42.6 mm to (162.3, 84.1), turned to -90 degrees
- moved J12 40.1 mm to (160.6, 79.8), turned to -90 degrees
- moved J11 40.1 mm to (160.6, 78.2), turned to -90 degrees
- moved C12 31.7 mm to (92.5, 87.7), turned to 180 degrees
- moved C10 24.7 mm to (95.9, 71.5), turned to 180 degrees
- moved C7 20.0 mm to (114.9, 82.5), turned to 180 degrees
- moved C1 17.7 mm to (107.8, 86.6)
- moved C11 15.8 mm to (110.5, 72.1), turned to 180 degrees
- moved Y1 14.8 mm to (113.2, 79.6), turned to -90 degrees
- moved C8 14.7 mm to (113.1, 76.5), turned to 0 degrees
- moved C13 13.0 mm to (89.7, 56.8), turned to 90 degrees
- moved U3 5.89 mm to (103.0, 78.1), turned to 180 degrees
- moved R6 4.80 mm to (138.0, 94.2), turned to -90 degrees
- moved REF** 2.57 mm to (83.2, 93.3)
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- renumbered C9 to C5, C5 to C6, C6 to C7, C7 to C8, C8 to C9, D4 to D2, D2 to D3, D3 to D4, J9 to J11, J10 to J12, J11 to J13, J6 to J9, R5 to R1, R1 to R5, R2 to R6
Connections:
- net USB_DM renamed USB_D-
- net USB_DP renamed USB_D+
- D4 pad 2: Net-(D3-Pad2) (its old number) -> Net-(D4-Pad2)
- J8 pad 1: unconnected-(J7-Pad1) -> +3V3
- J8 pad 10: unconnected-(J7-Pad10) -> Net-(J8-Pad10)
- J8 pad 11: unconnected-(J7-Pad11) -> Net-(J8-Pad11)
- J8 pad 12: unconnected-(J7-Pad12) -> Net-(J8-Pad12)
- J8 pad 13: unconnected-(J7-Pad13) -> Net-(J8-Pad13)
- J8 pad 14: unconnected-(J7-Pad14) -> Net-(J8-Pad14)
- J8 pad 15: unconnected-(J7-Pad15) -> Net-(J8-Pad15)
- J8 pad 16: unconnected-(J7-Pad16) -> Net-(J8-Pad16)
- J8 pad 17: unconnected-(J7-Pad17) -> Net-(J8-Pad17)
- J8 pad 18: unconnected-(J7-Pad18) -> Net-(J8-Pad18)
- J8 pad 19: unconnected-(J7-Pad19) -> Net-(J8-Pad19)
- J8 pad 2: unconnected-(J7-Pad2) -> GND
- J8 pad 20: unconnected-(J7-Pad20) -> LED_USR1
- J8 pad 3: unconnected-(J7-Pad3) -> SPI2_MISO
- J8 pad 4: unconnected-(J7-Pad4) -> SPI2_MOSI
- J8 pad 5: unconnected-(J7-Pad5) -> W5500_CS
- J8 pad 6: unconnected-(J7-Pad6) -> SPI2_SCK
- J8 pad 9: unconnected-(J7-Pad9) -> GND
- R3 pad 2: unconnected-(R3-Pad2) -> /USB_N
- R4 pad 2: unconnected-(R4-Pad2) -> /USB_P
- R5 pad 1: unconnected-(R1-Pad1) -> LED_USR1
- R6 pad 2: Net-(D3-Pad2) (its old number) -> Net-(J10-Pad2)
- U3 pad 14: unconnected-(U3-Pad14) -> LED_USR1
- U3 pad 15: unconnected-(U3-Pad15) -> Net-(J8-Pad19)
- U3 pad 16: unconnected-(U3-Pad16) -> Net-(J8-Pad18)
- U3 pad 17: unconnected-(U3-Pad17) -> Net-(J8-Pad17)
- U3 pad 20: unconnected-(U3-Pad20) -> Net-(J8-Pad16)
- U3 pad 21: unconnected-(U3-Pad21) -> Net-(J8-Pad15)
- U3 pad 22: unconnected-(U3-Pad22) -> Net-(J8-Pad14)
- U3 pad 23: unconnected-(U3-Pad23) -> Net-(J8-Pad13)
- U3 pad 41: unconnected-(U3-Pad41) -> Net-(J8-Pad12)
- U3 pad 42: unconnected-(U3-Pad42) -> Net-(J8-Pad11)
- U3 pad 43: unconnected-(U3-Pad43) -> Net-(J8-Pad10)
- U3 pad 44: unconnected-(U3-Pad44) -> /USB_N
- U3 pad 45: unconnected-(U3-Pad45) -> /USB_P
- U3 pad 48: unconnected-(U3-Pad48) -> +3V3
- U3 pad 60: unconnected-(U3-Pad60) -> Net-(R2-Pad2)
Routing:
- net +3V3: track 50.5 -> 134.7 mm, vias 1 -> 6
- net SPI2_MOSI: track 0.00 -> 42.7 mm
- net Net-(J8-Pad18): track 0.00 -> 34.9 mm, vias 0 -> 1
- net Net-(J8-Pad17): track 0.00 -> 34.6 mm, vias 0 -> 1
- net Net-(J8-Pad16): track 0.00 -> 33.4 mm, vias 0 -> 1
- net Net-(J8-Pad15): track 0.00 -> 32.6 mm, vias 0 -> 1
- net SWDIO: track 0.00 -> 30.7 mm
- net Net-(J8-Pad14): track 0.00 -> 30.6 mm, vias 0 -> 1
- net Net-(J8-Pad13): track 0.00 -> 29.9 mm, vias 0 -> 1
- net SWCLK: track 0.00 -> 25.2 mm
- net SPI2_MISO: track 0.00 -> 24.4 mm
- net GND: track 48.7 -> 72.8 mm, vias 88 -> 116
- net W5500_INT: track 0.00 -> 23.1 mm, vias 0 -> 1
- net /USB_N: track 0.00 -> 17.7 mm
- net Net-(J8-Pad10): track 0.00 -> 15.8 mm, vias 0 -> 1
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- added copper zone on In1.Cu, net GND
- added copper zone on In2.Cu, net GND
Other:
- copper layers 2 -> 4
- board text added: "+"
- board text added: "-"
- board text added: "2"
- board text added: "3"
- board text added: "4"
- board text added: "BATT."
- board text added: "BOOT"
- board text added: "BOTTOM"
- board text added: "L1 L2 L3 L4 L5"
- board text added: "PA0 USR1"
- board text added: "PROG"
- board text added: "RST"
- board text added: "SPI2_MISO"
- board text added: "SPI2_MOSI"
- board text added: "SPI2_SCK"
- board text added: "TOP"
- board text added: "U1 U2 U3 U4 U5"
- board text added: "W5500_CS"
- board text removed: "USR1"
- board text removed: "progr."
- board text removed: "tbd:5V IN->"

Commit message: save
Parts:
- added C10: 12p, Capacitor_SMD:C_0603_1608Metric, F.Cu at (114.0, 86.1)
- added C16: 22u, Capacitor_SMD:C_0805_2012Metric_Pad1.18x1.45mm_HandSolder, F.Cu at (128.3, 73.5)
- added C17: 22u, Capacitor_SMD:C_0805_2012Metric_Pad1.18x1.45mm_HandSolder, F.Cu at (126.2, 73.5)
- added C18: 100n, Capacitor_SMD:C_0805_2012Metric, F.Cu at (126.2, 78.4)
- added C9: 12p, Capacitor_SMD:C_0603_1608Metric, F.Cu at (111.5, 86.1)
- added J15: Micro_SD_Card, Connector_Card:microSD_HC_Hirose_DM3BT-DSF-PEJS, F.Cu at (142.7, 77.2)
- added R10: 10k, Resistor_SMD:R_0603_1608Metric_Pad0.98x0.95mm_HandSolder, F.Cu at (130.2, 73.7)
- added R11: 10k, Resistor_SMD:R_0603_1608Metric_Pad0.98x0.95mm_HandSolder, F.Cu at (130.2, 77.2)
- added R7: 10k, Resistor_SMD:R_0603_1608Metric_Pad0.98x0.95mm_HandSolder, F.Cu at (128.6, 79.0)
- added R8: 10k, Resistor_SMD:R_0603_1608Metric_Pad0.98x0.95mm_HandSolder, F.Cu at (131.8, 74.2)
- added R9: 10k, Resistor_SMD:R_0603_1608Metric_Pad0.98x0.95mm_HandSolder, F.Cu at (131.8, 77.6)
- added Y2: 32.768k, Crystal:Crystal_SMD_3215-2Pin_3.2x1.5mm, F.Cu at (112.7, 83.3)
- moved R5 1.96 mm to (139.8, 60.0), turned to -90 degrees
- moved C7 1.88 mm to (116.8, 82.5)
- moved C8 1.88 mm to (115.0, 76.5)
- moved Y1 1.88 mm to (115.1, 79.5)
- moved J3 0.40 mm to (85.8, 100.8)
- renumbered C9 to C11, C10 to C12, C11 to C13, C12 to C14, C13 to C15
Connections:
- J8 pad 3: SPI2_MISO -> unconnected-(J8-Pad3)
- J8 pad 4: SPI2_MOSI -> unconnected-(J8-Pad4)
- J8 pad 5: W5500_CS -> unconnected-(J8-Pad5)
- J8 pad 6: SPI2_SCK -> unconnected-(J8-Pad6)
- U3 pad 3: unconnected-(U3-Pad3) -> Net-(C9-Pad2)
- U3 pad 39: unconnected-(U3-Pad39) -> SDMMC1_D0
- U3 pad 4: unconnected-(U3-Pad4) -> Net-(C10-Pad2)
- U3 pad 40: unconnected-(U3-Pad40) -> SDMMC1_D1
- U3 pad 51: unconnected-(U3-Pad51) -> SDMMC1_D2
- U3 pad 52: unconnected-(U3-Pad52) -> SDMMC1_D3
- U3 pad 53: unconnected-(U3-Pad53) -> SDMMC1_CLK
- U3 pad 54: unconnected-(U3-Pad54) -> SDMMC1_CMD
Routing:
- net +3V3: track 134.7 -> 209.0 mm, vias 6 -> 8
- net SDMMC1_CMD: track 0.00 -> 48.1 mm, vias 0 -> 2
- net SDMMC1_CLK: track 0.00 -> 46.4 mm, vias 0 -> 2
- net SDMMC1_D3: track 0.00 -> 45.6 mm, vias 0 -> 2
- net LED_USR1: track 0.83 -> 45.2 mm, vias 0 -> 1
- net SDMMC1_D2: track 0.00 -> 40.1 mm, vias 0 -> 2
- net Net-(J8-Pad19): track 0.73 -> 38.8 mm, vias 0 -> 1
- net Net-(J8-Pad12): track 6.42 -> 39.7 mm
- net Net-(J8-Pad11): track 9.59 -> 41.1 mm
- net Net-(J8-Pad10): track 15.8 -> 45.4 mm
- net SPI2_MOSI: track 42.7 -> 17.0 mm
- net SPI2_SCK: track 15.2 -> 40.6 mm
- net GND: track 72.8 -> 94.0 mm, vias 116 -> 127
- net W5500_CS: track 11.7 -> 23.6 mm
- net Net-(C10-Pad2): track 0.00 -> 8.49 mm
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Other:
- board text added: "16 MHz + 32.768 kHz crystals"
- board text added: "gnd"
- board text added: "microSD"
- board text removed: "16MHz"
- board text removed: "L1 L2 L3 L4 L5"
- board text removed: "SPI2_MISO"
- board text removed: "SPI2_MOSI"
- board text removed: "SPI2_SCK"
- board text removed: "U1 U2 U3 U4 U5"
- board text removed: "W5500_CS"

Commit message: save
Parts:
- removed the J14 at (93.0, 100.7)
- removed the J15 at (142.7, 77.2)
- added J10: Conn_02x16_Odd_Even, Connector_PinHeader_2.54mm:PinHeader_2x16_P2.54mm_Vertical, F.Cu at (87.8, 57.2)
- added J16: SD_Card, Connector_Card:SD_Kyocera_145638109211859+, B.Cu at (127.0, 79.0)
- added J6: Conn_02x05_Odd_Even, Connector_IDC:IDC-Header_2x05_P2.54mm_Vertical, F.Cu at (93.9, 98.8)
- H1, H2, H3, H4: footprint MountingHole:MountingHole_2.7mm_M2.5_DIN965_Pad -> MountingHole:MountingHole_3.2mm_M3_DIN965_Pad_TopBottom
- J9: renamed from J8; value upper_header -> long_header
- moved D3 38.8 mm to (150.2, 99.6), turned to 90 degrees
- moved R5 36.9 mm to (145.2, 96.6), turned to 0 degrees
- moved JP1 35.9 mm to (148.9, 96.3)
- moved J11 34.8 mm to (147.2, 99.5)
- moved J9 31.6 mm to (76.5, 28.8)
- moved J12 30.2 mm to (173.7, 91.4)
- moved JP2 30.2 mm to (171.8, 95.2)
- moved D4 30.2 mm to (176.3, 95.2)
- moved R6 30.2 mm to (168.3, 94.2)
- moved J3 25.9 mm to (76.4, 124.9)
- moved R7 17.3 mm to (115.3, 67.9), turned to 0 degrees
- moved C15 13.4 mm to (76.3, 57.1)
- moved J8 13.0 mm to (112.5, 100.7), turned to 180 degrees
- moved R8 11.5 mm to (121.7, 79.7), turned to -90 degrees
- moved H3 11.0 mm to (136.2, 55.9)
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- renumbered J9 to J11, J10 to J12, J11 to J13, J12 to J14, J13 to J15, J6 to J7, J7 to J8
Routing:
- net +3V3: track 209.0 -> 152.0 mm, vias 8 -> 6
- net SDMMC1_CMD: track 48.1 -> 20.9 mm
- net SDMMC1_CLK: track 46.4 -> 25.0 mm
- net SWDIO: track 31.1 -> 11.1 mm
- net SPI2_SCK: track 40.6 -> 20.8 mm, vias 2 -> 1
- net LED_USR1: track 45.2 -> 25.8 mm
- net SDMMC1_D2: track 40.1 -> 20.8 mm, vias 2 -> 1
- net RST: track 81.9 -> 63.4 mm
- net SDMMC1_D3: track 45.6 -> 27.8 mm
- net GND: track 94.0 -> 76.3 mm, vias 127 -> 109
- net Net-(J9-Pad19): track 38.8 -> 21.9 mm
- net Net-(J9-Pad16): track 33.4 -> 16.9 mm
- net Net-(J9-Pad18): track 34.8 -> 18.4 mm
- net Net-(J9-Pad17): track 34.7 -> 18.6 mm
- net Net-(J9-Pad13): track 29.8 -> 14.0 mm
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Other:
- board size 84.9 x 52.9 mm -> 73.6 x 52.9 mm
- board text added: "BOOT SEL."
- board text added: "DC IN"
- board text added: "PA0"
- board text added: "RJ45 keepout area"
- board text added: "STLINK2 PROGR."
- board text added: "USR LED"
- board text removed: "BATT."
- board text removed: "BOOT"
- board text removed: "PA0 USR1"
- board text removed: "PROG"
- board text removed: "W5500 module"
- board text removed: "microSD"

Commit message: save
Routing:
- net GND: track 76.3 -> 78.3 mm
Other:
- board text added: "A1"
- board text added: "SD card"
- board text removed: "STM32L475"
- board text removed: "gnd"
Changed lines of the file:
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@@
     (pad "32" thru_hole oval (at 2.54 38.1 90) (size 1.7 1.7) (drill 1) (layers *.Cu *.Mask)
       (net 1 "GND") (pinfunction "Pin_32") (pintype "passive"))
-    (model "${KICAD6_3DMODEL_DIR}/Connector_PinHeader_2.54mm.3dshapes/PinHeader_2x16_P2.54mm_Vertical.wrl" hide
+    (model "${KICAD6_3DMODEL_DIR}/Connector_PinHeader_2.54mm.3dshapes/PinHeader_2x16_P2.54mm_Vertical.wrl"
       (offset (xyz 0 0 0))
       (scale (xyz 1 1 1))
@@
     )
   )
+  (gr_rect (start 86.4 52.125) (end 127.4 55.875) (layer "B.SilkS") (width 0.2) (fill solid))
+  (gr_line (start 91.15 42.975) (end 131 42.875) (layer "B.SilkS") (width 1))
   (gr_line (start 75.192 61.505) (end 76.081 61.505) (layer "F.SilkS") (width 0.4))
   (gr_circle (center 135.8 62.75) (end 136.992686 62.75) (layer "F.SilkS") (width 0.5) (fill none))
   (gr_rect (start 83.15 60.325) (end 138.15 88.475) (layer "F.SilkS") (width 0.5) (fill none))
   (gr_circle (center 75.7 64.172) (end 76.716 64.172) (layer "F.SilkS") (width 0.2) (fill none))
+  (gr_line (start 87.05 52.775) (end 126.9 52.875) (layer "F.SilkS") (width 1))
   (gr_circle (center 135.825 86.125) (end 137.017686 86.125) (layer "F.SilkS") (width 0.5) (fill none))
   (gr_rect (start 138.1 66.125) (end 114.2 83.325) (layer "F.SilkS") (width 0.5) (fill none))
@@
     (effects (font (size 1.5 1.5) (thickness 0.375)) (justify mirror))
   )
-  (gr_text "STM32L475" (at 101.175 91.725) (layer "B.SilkS")
-    (effects (font (size 2.5 2.5) (thickness 0.625)) (justify mirror))
+  (gr_text "MCU: STM32L475RCTx" (at 115 64.275) (layer "B.SilkS")
+    (effects (font (size 1.5 1.5) (thickness 0.375)) (justify mirror))
+  )
+  (gr_text "GND" (at 128.45 54.075 90) (layer "B.SilkS")
+    (effects (font (size 1 1) (thickness 0.25)) (justify mirror))
+  )
+  (gr_text "3V3" (at 87.78211 59.400212) (layer "B.SilkS")
+    (effects (font (size 1 0.8) (thickness 0.2)) (justify mirror))
+  )
+  (gr_text "GND" (at 84.8 53.925 90) (layer "B.SilkS")
+    (effects (font (size 1 1) (thickness 0.25)) (justify mirror))
   )
   (gr_text "ELECTROSTATIC\nSENSITIVE\nDEVICES" (at 78 69.025) (layer "B.SilkS")
     (effects (font (size 1 1) (thickness 0.25)) (justify mirror))
   )
+  (gr_text "SD card" (at 124.5 95.125) (layer "B.SilkS")
+    (effects (font (size 1.5 1.5) (thickness 0.375)) (justify mirror))
+  )
   (gr_text "3V3" (at 88.1 90.4) (layer "F.SilkS")
     (effects (font (size 1 1) (thickness 0.25)))
@@
     (effects (font (size 1 1) (thickness 0.25)))
   )
-  (gr_text "gnd" (at 82.085 53.345) (layer "F.SilkS")
-    (effects (font (size 1 1) (thickness 0.25)))
-  )
   (gr_text "D+" (at 76.9 79.4 90) (layer "F.SilkS")
     (effects (font (size 1 1) (thickness 0.25)))
@@
     (effects (font (size 1 1) (thickness 0.25)))
   )
+  (gr_text "GND" (at 84.7 54.125 90) (layer "F.SilkS")
+    (effects (font (size 1 1) (thickness 0.25)))
+  )
   (gr_text "TODO: KAIKKI MITAT \nRASTERIJAKOON!" (at 113.8174 36.957) (layer "F.SilkS")
     (effects (font (size 2 2) (thickness 0.5)))
@@
     (effects (font (size 1 1) (thickness 0.25)))
   )
-  (gr_text "3V3" (at 92.7862 59.182 90) (layer "F.SilkS")
-    (effects (font (size 1 1) (thickness 0.25)))
-  )
   (gr_text "+" (at 76.632 127.345) (layer "F.SilkS")
     (effects (font (size 1 1) (thickness 0.25)))
@@
     (effects (font (size 1 1) (thickness 0.25)))
   )
-  (gr_text "GND" (at 99.665 58.9952 90) (layer "F.SilkS")
-    (effects (font (size 1 1) (thickness 0.25)))
-  )
   (gr_text "NC" (at 82.65 72.59) (layer "F.SilkS")
     (effects (font (size 1 1) (thickness 0.25)))
@@
     (effects (font (size 1 1) (thickness 0.25)))
   )
-  (gr_text "GND" (at 81.9358 59.5032 90) (layer "F.SilkS")
-    (effects (font (size 1 1) (thickness 0.25)))
-  )
   (gr_text "RST" (at 82.44 67.486) (layer "F.SilkS")
     (effects (font (size 1 1) (thickness 0.25)))
   )
+  (gr_text "3V3" (at 87.8 59.425) (layer "F.SilkS")
+    (effects (font (size 1 0.8) (thickness 0.2)))
+  )
+  (gr_text "GND" (at 128.5 54.225 90) (layer "F.SilkS")
+    (effects (font (size 1 1) (thickness 0.25)))
+  )
   (gr_text "SCK" (at 91.1 72.665) (layer "F.SilkS")
     (effects (font (size 1 1) (thickness 0.25)))
@@
   (gr_text "BOOT SEL." (at 115.05 98.025 90) (layer "F.SilkS")
     (effects (font (size 1 1) (thickness 0.25)))
+  )
+  (gr_text "A1" (at 100.5 59.425) (layer "F.SilkS")
+    (effects (font (size 1 0.8) (thickness 0.2)))
   )
   (gr_text "STLINK2\nPROGR." (at 84.25 100.575) (layer "F.SilkS")
@@
   (segment (start 110.0414 86.5994) (end 110.0668 86.6248) (width 1) (layer "F.Cu") (net 1))
   (segment (start 100.3822 74.525) (end 99.7916 73.9344) (width 0.3) (layer "F.Cu") (net 1))
+  (segment (start 87.75 54.635) (end 85.79 54.635) (width 1) (layer "F.Cu") (net 1))
   (segment (start 104.9 76.95) (end 105.3 76.55) (width 0.3) (layer "F.Cu") (net 1))
   (segment (start 99.5004 80.3764) (end 98.5684 81.3084) (width 0.3) (layer "F.Cu") (net 1))
@@
   (segment (start 116.725 78.45) (end 115.975 78.45) (width 1) (layer "F.Cu") (net 1))
   (segment (start 86.4616 95.9866) (end 85.9628 95.9866) (width 1) (layer "F.Cu") (net 1))
+  (segment (start 85.79 54.635) (end 85.75 54.675) (width 1) (layer "F.Cu") (net 1))
   (segment (start 106.2916 72.3834) (end 106.2916 74.1754) (width 0.3) (layer "F.Cu") (net 1))
   (segment (start 150.175 100.525) (end 150.175 101.8) (width 1) (layer "F.Cu") (net 1))

Commit message: save
Parts:
- removed J13, J14: Conn_01x01_Female, Connector_Wire:SolderWirePad_1x01_SMD_1x2mm
- removed the J15 at (162.3, 84.1)
- removed the J7 at (71.1, 64.3)
- removed the J9 at (76.5, 28.8)
- added C1: 100u, Capacitor_SMD:C_0805_2012Metric, F.Cu at (77.0, 103.1)
- added C3: 100n, Capacitor_SMD:C_0805_2012Metric, F.Cu at (84.3, 103.0)
- added D1: SS34, Diode_SMD:D_SMA, F.Cu at (81.3, 100.2)
- added F2: 630mA, Resistor_THT:R_Axial_DIN0207_L6.3mm_D2.5mm_P7.62mm_Horizontal, F.Cu at (80.6, 72.7)
- J3: value STLINK -> DCin; footprint Connector_PinHeader_2.54mm:PinHeader_1x04_P2.54mm_Vertical -> Connector_BarrelJack:BarrelJack_Horizontal
- J6: value Conn_02x05_Odd_Even -> STLINK2
- R1: value 2k -> 1.5k
- moved J3 59.8 mm to (77.0, 65.1), turned to 0 degrees
- moved D3 53.7 mm to (117.2, 96.4), turned to -90 degrees
- moved R1 52.5 mm to (117.2, 99.9), turned to 90 degrees
- moved J11 32.9 mm to (149.3, 113.5)
- moved JP2 32.9 mm to (147.4, 117.3)
- moved D5 32.9 mm to (151.9, 117.3)
- moved R6 32.9 mm to (143.9, 116.2)
- moved C18 26.0 mm to (107.8, 90.7), turned to 90 degrees
- moved C19 23.2 mm to (109.8, 90.7), turned to 90 degrees
- moved R7 20.0 mm to (115.8, 87.9), turned to -90 degrees
- moved REF** 16.1 mm to (83.5, 77.3)
- moved R10 15.3 mm to (113.2, 90.6)
- moved R9 15.0 mm to (121.0, 87.9), turned to -90 degrees
- moved R11 13.6 mm to (119.5, 87.9), turned to -90 degrees
- moved C20 12.5 mm to (117.6, 88.0), turned to -90 degrees
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- renumbered C8 to C10, C9 to C11, C10 to C12, C11 to C13, C12 to C14, C13 to C15, C14 to C16, C15 to C17, C16 to C18, C17 to C19, C1 to C2, C18 to C20, C3 to C5, C4 to C6, C5 to C7, C6 to C8, C7 to C9, D1 to D2, D2 to D3, D3 to D4, D4 to D5, J11 to J10, J12 to J11, J16 to J15, J8 to J7, J10 to J9
Connections:
- J3 pad 1: +3V3 -> Net-(F2-Pad2)
- J3 pad 2: SWCLK -> GND
- J3 pad 3: SWDIO -> (no net)
- J6 pad 1: unconnected-(J6-Pad1) -> RST
- J6 pad 2: unconnected-(J6-Pad2) -> SWDIO
- J6 pad 3: unconnected-(J6-Pad3) -> GND
- J6 pad 4: unconnected-(J6-Pad4) -> GND
- J6 pad 6: unconnected-(J6-Pad6) -> SWCLK
- J6 pad 7: unconnected-(J6-Pad7) -> +3V3
- J6 pad 8: unconnected-(J6-Pad8) -> +3V3
- R1 pad 1: VBUS -> +3V3
- U3 pad 15: Net-(J9-Pad19) -> unconnected-(U3-Pad15)
- U3 pad 16: Net-(J9-Pad18) -> unconnected-(U3-Pad16)
- U3 pad 17: Net-(J9-Pad17) -> unconnected-(U3-Pad17)
- U3 pad 20: Net-(J9-Pad16) -> unconnected-(U3-Pad20)
- U3 pad 21: Net-(J9-Pad15) -> unconnected-(U3-Pad21)
- U3 pad 22: Net-(J9-Pad14) -> unconnected-(U3-Pad22)
- U3 pad 23: Net-(J9-Pad13) -> unconnected-(U3-Pad23)
- U3 pad 41: Net-(J9-Pad12) -> unconnected-(U3-Pad41)
- U3 pad 42: Net-(J9-Pad11) -> unconnected-(U3-Pad42)
- U3 pad 43: Net-(J9-Pad10) -> unconnected-(U3-Pad43)
Routing:
- net +3V3: track 152.0 -> 190.6 mm, vias 6 -> 5
- net Net-(C1-Pad1): track 0.00 -> 37.0 mm, vias 0 -> 1
- net unconnected-(U3-Pad43): track 0.00 -> 33.2 mm, vias 0 -> 1
- net Net-(J9-Pad10): track 33.2 -> 0.00 mm, vias 1 -> 0
- net unconnected-(U3-Pad42): track 0.00 -> 32.3 mm, vias 0 -> 1
- net Net-(J9-Pad11): track 32.3 -> 0.00 mm, vias 1 -> 0
- net GND: track 78.3 -> 106.1 mm, vias 109 -> 119
- net unconnected-(U3-Pad41): track 0.00 -> 25.0 mm, vias 0 -> 1
- net Net-(J9-Pad12): track 25.0 -> 0.00 mm, vias 1 -> 0
- net unconnected-(U3-Pad15): track 0.00 -> 21.9 mm, vias 0 -> 1
- net Net-(J9-Pad19): track 21.9 -> 0.00 mm, vias 1 -> 0
- net LED_USR1: track 25.8 -> 4.32 mm
- net unconnected-(U3-Pad17): track 0.00 -> 18.6 mm, vias 0 -> 1
- net Net-(J9-Pad17): track 18.6 -> 0.00 mm, vias 1 -> 0
- net unconnected-(U3-Pad16): track 0.00 -> 18.4 mm, vias 0 -> 1
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Other:
- board text added: "5..12V DC IN center +"
- board text added: "BOOT0"
- board text added: "DC_IN"
- board text added: "PWR LED"
- board text added: "STM32 PROGR."
- board text added: "SWCLK"
- board text added: "SWDIO"
- board text added: "[PINOUT PIN-PER-PIN WILL BE HERE]"
- board text added: "barrel"
- board text added: "usb"
- board text removed: "+"
- board text removed: "-"
- board text removed: "CLK"
- board text removed: "DC IN"
- board text removed: "DIO"
- board text removed: "STLINK2 PROGR."
