File: STM32L475-protoboard.kicad_pcb (KiCad board)
At the start: 4 copper layers, 73.6 x 52.9 mm, 63 parts, among them J1 USB_HEADER, J10 Conn_01x02_Male, J11 Conn_01x02_Male, J15 SD_Card, J2 USB_B_Micro, J3 DCin, J5 W5500_ETHERNET, J6 STLINK2, J7 BOOT_MODE, J9 Conn_02x16_Odd_Even, SW1 RESET, U1 SRV05-4, U2 AMS1117-3.3, U3 STM32L475RCTx, Y1 Crystal_GND24, Y2 32.768k

Commit message: save
Parts:
- added C4: 100u, Capacitor_SMD:C_0805_2012Metric_Pad1.18x1.45mm_HandSolder, F.Cu at (84.9, 97.5)
- added C5: 100u, Capacitor_SMD:C_0805_2012Metric_Pad1.18x1.45mm_HandSolder, F.Cu at (80.6, 103.1)
- added R5: 1.5k, Resistor_SMD:R_0603_1608Metric_Pad0.98x0.95mm_HandSolder, F.Cu at (78.5, 81.8)
- J8: renamed from J9; value Conn_02x16_Odd_Even -> Conn_02x20_Odd_Even; footprint Connector_PinHeader_2.54mm:PinHeader_2x16_P2.54mm_Vertical -> Connector_PinHeader_2.54mm:PinHeader_2x20_P2.54mm_Vertical
- R1: footprint Resistor_SMD:R_0603_1608Metric -> Resistor_SMD:R_0603_1608Metric_Pad0.98x0.95mm_HandSolder
- R3, R4: value 0 -> 22; footprint Resistor_SMD:R_0805_2012Metric_Pad1.20x1.40mm_HandSolder -> Resistor_SMD:R_0603_1608Metric_Pad0.98x0.95mm_HandSolder
- R6: renamed from R5; footprint Resistor_SMD:R_0805_2012Metric_Pad1.20x1.40mm_HandSolder -> Resistor_SMD:R_0603_1608Metric_Pad0.98x0.95mm_HandSolder
- R7: renamed from R6; footprint Resistor_SMD:R_0805_2012Metric_Pad1.20x1.40mm_HandSolder -> Resistor_SMD:R_0603_1608Metric_Pad0.98x0.95mm_HandSolder
- moved C7 10.4 mm to (92.0, 63.4), turned to 180 degrees
- moved J8 6.60 mm to (81.2, 57.2)
- moved C9 2.41 mm to (80.8, 62.2)
- moved C1 1.35 mm to (76.1, 102.0), turned to -90 degrees
- moved C6 0.54 mm to (85.1, 95.5)
- moved C8 0.39 mm to (85.1, 93.5)
- moved C3 0.10 mm to (84.3, 103.1)
- moved D1 0.08 mm to (81.3, 100.3)
- renumbered C8 to C10, C9 to C11, C10 to C12, C11 to C13, C12 to C14, C13 to C15, C14 to C16, C15 to C17, C16 to C18, C18 to C19, C19 to C20, C20 to C21, C5 to C6, C17 to C7, C6 to C8, C7 to C9, J11 to J10, J15 to J11, J10 to J9, R9 to R10, R10 to R11, R11 to R12, R7 to R8, R8 to R9
Connections:
- C1 pad 1: Net-(C1-Pad1) -> +VDC
- D1 pad 2: Net-(C1-Pad1) -> +VDC
- F2 pad 1: Net-(C1-Pad1) -> +VDC
- J2 pad 4: unconnected-(J2-Pad4) -> /USB_ID
- J8 pad 1: +3V3 -> +VDC
- J8 pad 3: unconnected-(J9-Pad3) -> VBUS
- J8 pad 5: unconnected-(J9-Pad5) -> +3V3
- U3 pad 43: unconnected-(U3-Pad43) -> /USB_ID
Routing:
- net GND: track 106.1 -> 194.4 mm, vias 119 -> 120
- net Net-(C1-Pad1): track 37.0 -> 0.00 mm, vias 1 -> 0
- net +VDC: track 0.00 -> 36.6 mm, vias 0 -> 1
- net unconnected-(U3-Pad43): track 33.2 -> 0.00 mm, vias 1 -> 0
- net RST: track 69.0 -> 98.6 mm
- net VBUS: track 24.7 -> 44.1 mm
- net /USB_ID: track 0.00 -> 12.6 mm, vias 0 -> 1
- net +3V3: track 190.6 -> 180.4 mm, vias 5 -> 4
- net Net-(C3-Pad1): track 14.9 -> 17.2 mm
- net USB_D+: track 11.1 -> 13.0 mm
Other:
- board text added: "Vin"
- board text removed: "barrel"
- board text removed: "usb"

Commit message: saveä
Parts:
- added H5: MountingHole_Pad, MountingHole:MountingHole_2.2mm_M2_DIN965_Pad_TopBottom, F.Cu at (138.2, 62.6)
- moved D5 27.4 mm to (130.4, 100.2), turned to 90 degrees
- moved J9 26.7 mm to (120.6, 99.5), turned to 180 degrees
- moved R7 26.6 mm to (130.4, 93.3)
- moved JP2 26.6 mm to (130.4, 96.8), turned to -90 degrees
- moved D4 26.4 mm to (123.8, 100.2)
- moved J10 26.1 mm to (127.2, 99.5), turned to 180 degrees
- moved JP1 25.1 mm to (123.8, 96.8), turned to -90 degrees
- moved R6 21.6 mm to (123.8, 93.3), turned to -90 degrees
- moved C11 1.97 mm to (115.0, 83.5), turned to 90 degrees
- moved TP1 1.29 mm to (87.7, 89.4)
- moved C12 0.67 mm to (114.4, 76.6)
- moved C14 0.65 mm to (113.3, 86.1)
- moved Y2 0.65 mm to (112.0, 83.3)
- moved Y1 0.58 mm to (114.5, 79.5)
Connections:
- J8 pad 37: unconnected-(J8-Pad37) -> LED_USR1
- J8 pad 39: unconnected-(J8-Pad39) -> LED_USR2
- R7 pad 1: unconnected-(R7-Pad1) -> LED_USR2
- U3 pad 15: unconnected-(U3-Pad15) -> LED_USR2
Routing:
- net LED_USR2: track 0.00 -> 56.8 mm, vias 0 -> 3
- net LED_USR1: track 4.32 -> 52.5 mm, vias 1 -> 3
- net SDMMC1_D3: track 28.9 -> 53.0 mm, vias 2 -> 3
- net unconnected-(U3-Pad15): track 21.9 -> 0.00 mm, vias 1 -> 0
- net unconnected-(U3-Pad16): track 18.4 -> 2.76 mm
- net SDMMC1_CMD: track 23.0 -> 35.7 mm
- net unconnected-(U3-Pad17): track 18.6 -> 8.16 mm
- net unconnected-(U3-Pad20): track 16.9 -> 10.5 mm
- net SDMMC1_D1: track 5.26 -> 11.4 mm, vias 1 -> 2
- net SDMMC1_D2: track 22.7 -> 28.8 mm
- net SDMMC1_CLK: track 23.6 -> 18.7 mm
- net Net-(J10-Pad2): track 2.51 -> 5.42 mm
- net +3V3: track 180.4 -> 182.8 mm
- net SDMMC1_D0: track 8.51 -> 10.9 mm, vias 1 -> 2
- net Net-(J9-Pad2): track 3.51 -> 5.54 mm
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Other:
- board text added: "LL'23"
- board text added: "PA1"
- board text added: "PWR"
- board text added: "RJ45 keepout"
- board text added: "USR1"
- board text added: "pin 1"
- board text removed: "OH3HZB 2023"
- board text removed: "PWR LED"
- board text removed: "RJ45 keepout area"
- board text removed: "USR LED"
